Commit message: Backup

File: group4/src/hippo2/defs/pioneer3dx.xacro (robot description, xacro)
@@ -2,5 +2,5 @@
 <robot name="pioneer3dx"
 	xmlns:xacro="http://ros.org/wiki/xacro">
-  <include filename="$(find p2os_urdf)/defs/pioneer3dx_wheel.xacro"/>
+  <include filename="$(find hippo2)/defs/pioneer3dx_wheel.xacro"/>
 <!-- Chassis -->
 	<link name="base_link">
@@ -16,5 +16,5 @@
 			<origin xyz="-0.045 0 0.148" rpy="0 0 0"/>
 			<geometry name="pioneer_geom">
-				<mesh filename="package://p2os_urdf/meshes/p3dx_meshes/chassis.stl"/>
+				<mesh filename="package://hippo2/meshes/p3dx_meshes/chassis.stl"/>
 			</geometry>
 			<material name="ChassisRed">
@@ -41,5 +41,5 @@
 			<origin xyz="0 0 0" rpy="0 0 0"/>
 			<geometry name="top_geom">
-				<mesh filename="package://p2os_urdf/meshes/p3dx_meshes/top.stl"/>
+				<mesh filename="package://hippo2/meshes/p3dx_meshes/top.stl"/>
 			</geometry>
 			<material name="TopBlack">
@@ -70,5 +70,5 @@
 		<origin xyz="0 0 0" rpy="0 0 0"/>
 		<geometry name="pioneer_geom">
-			<mesh filename="package://p2os_urdf/meshes/p3dx_meshes/swivel.stl"/>
+			<mesh filename="package://hippo2/meshes/p3dx_meshes/swivel.stl"/>
 		</geometry>
 		<material name="swivel">
@@ -103,5 +103,5 @@
 		<origin xyz="0 0 0" rpy="0 0 0"/>
 		<geometry name="pioneer_geom">
-			<mesh filename="package://p2os_urdf/meshes/p3dx_meshes/center_hubcap.stl"/>
+			<mesh filename="package://hippo2/meshes/p3dx_meshes/center_hubcap.stl"/>
 		</geometry>
 		<material name="swivel">
@@ -135,5 +135,5 @@
 		<origin xyz="0 0 0" rpy="0 0 0"/>
 		<geometry name="pioneer_geom">
-			<mesh filename="package://p2os_urdf/meshes/p3dx_meshes/center_wheel.stl"/>
+			<mesh filename="package://hippo2/meshes/p3dx_meshes/center_wheel.stl"/>
 		</geometry>
 		<material name="WheelBlack">
@@ -144,5 +144,5 @@
 		<origin xyz="0 0 0" rpy="${-3.1415927/2.0} 0 0"/>
 		<geometry>
-			<!--<mesh filename="package://p2os_urdf/meshes/p3dx_meshes/center_wheel.stl"/>-->
+			<!--<mesh filename="package://hippo2/meshes/p3dx_meshes/center_wheel.stl"/>-->
 			<cylinder radius="0.0375" length="0.01"/>
 		</geometry>
@@ -167,5 +167,5 @@
 			<origin xyz="0 0 0" rpy="0 0 0"/>
 			<geometry name="pioneer_geom">
-				<mesh filename="package://p2os_urdf/meshes/p3dx_meshes/front_sonar.stl"/>
+				<mesh filename="package://hippo2/meshes/p3dx_meshes/front_sonar.stl"/>
 			</geometry>
 			<material name="SonarYellow">
@@ -195,5 +195,5 @@
 			<origin xyz="0 0 0" rpy="0 0 0"/>
 			<geometry name="pioneer_geom">
-				<mesh filename="package://p2os_urdf/meshes/p3dx_meshes/back_sonar.stl"/>
+				<mesh filename="package://hippo2/meshes/p3dx_meshes/back_sonar.stl"/>
 			</geometry>
 			<material name="SonarYellow">
@@ -245,8 +245,7 @@
  <!-- Camera -->
 	<joint name="servo_joint" type="fixed">
-	  <parent link="base_link"/>
+	  <parent link="top_plate"/>
 	  <child link="camera_y_link"/>
-	  <origin xyz="13 0 0" rpy="0 0 0"/>
-	  <axis xyz="0 0 1"/>
+	  <origin xyz="0.13 0 0" rpy="0 0 0"/>
   </joint>
 	<link name="camera_y_link"/>
@@ -254,6 +253,6 @@
 	  <parent link="camera_y_link"/>
 	  <child link="camera_z_link"/>
-	  <origin xyz="0 6 0" rpy="0 90 0"/>continuous
-	  <axis xyz="0 1 0"/>
+	  <origin xyz="0 0 0.06" rpy="0 0 4.25"/>
+	  <axis xyz="0 0 1"/>
   </joint>
 	<link name="camera_z_link"/>
@@ -261,11 +260,11 @@
 	  <parent link="camera_z_link"/>
 	  <child link="camera_link"/>
-	  <origin xyz="0 3 0" rpy="0 0 90"/>
-	  <axis xyz="0 0 1"/>
+	  <origin xyz="0 0 0.03" rpy="0 1.57 0"/>
+	  <axis xyz="0 1 0"/>
 	</joint>
 	<!-- this should be camera link -->
 	<link name="camera_link">
 	  <inertia>
-	    <origin xyz="0 0 7"/>
+	    <origin xyz="0 0 0.07"/>
     </inertia>
 	</link>

Commit message: point2laser

File: group4/src/hippo2/defs/pioneer3dx.xacro (robot description, xacro)
@@ -260,5 +260,5 @@
 	  <parent link="camera_z_link"/>
 	  <child link="camera_link"/>
-	  <origin xyz="0 0 0.03" rpy="0 1.57 0"/>
+	  <origin xyz="0 0 0.09" rpy="0 4.7128 0"/>
 	  <axis xyz="0 1 0"/>
 	</joint>

Commit message: backup

File: group4/src/hippo2/defs/pioneer3dx.xacro (robot description, xacro)
@@ -253,5 +253,5 @@
 	  <parent link="camera_y_link"/>
 	  <child link="camera_z_link"/>
-	  <origin xyz="0 0 0.06" rpy="0 0 4.25"/>
+	  <origin xyz="0 0 0.06" rpy="0 0 4.35"/> <!--0 0 4.25-->
 	  <axis xyz="0 0 1"/>
   </joint>
@@ -260,12 +260,8 @@
 	  <parent link="camera_z_link"/>
 	  <child link="camera_link"/>
-	  <origin xyz="0 0 0.09" rpy="0 4.7128 0"/>
+	  <origin xyz="0 0 0.09" rpy="0 4.65 0"/>
 	  <axis xyz="0 1 0"/>
 	</joint>
 	<!-- this should be camera link -->
-	<link name="camera_link">
-	  <inertia>
-	    <origin xyz="0 0 0.07"/>
-    </inertia>
-	</link>
+	<link name="camera_link"/>
 </robot>
